File: design/Power.kicad_sch (KiCad schematic)
At the start: 48 parts, among them U2 TC2117, U3 DRV8302

Commit message: Limpando warnings e DRC errors
Parts:
- C25, C33: footprint w_smd_cap:c_tant_B -> CRF1:c_tant_B
- C39: footprint CRF1:SMD-1206 -> Capacitor_SMD:C_1206_3216Metric_Pad1.33x1.80mm_HandSolder
- C51: footprint w_smd_cap:c_2220 -> CRF1:c_2220
- D5: footprint w_smd_diode:do214ac -> CRF1:do214ac
- U2: footprint CRF1:SOT-223 -> Package_TO_SOT_SMD:SOT-223
Changed lines of the file:
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@@
       (effects (font (size 1.27 1.27)) (justify left))
     )
-    (property "Footprint" "w_smd_cap:c_tant_B" (at 222.25 82.55 0)
+    (property "Footprint" "CRF1:c_tant_B" (at 222.25 82.55 0)
       (effects (font (size 1.524 1.524)) hide)
     )
@@
       (effects (font (size 1.27 1.27)) (justify left))
     )
-    (property "Footprint" "w_smd_cap:c_tant_B" (at 182.88 35.56 0)
+    (property "Footprint" "CRF1:c_tant_B" (at 182.88 35.56 0)
       (effects (font (size 1.524 1.524)) hide)
     )
@@
       (effects (font (size 1.27 1.27)) (justify left))
     )
-    (property "Footprint" "CRF1:SMD-1206" (at 184.15 71.12 0)
+    (property "Footprint" "Capacitor_SMD:C_1206_3216Metric_Pad1.33x1.80mm_HandSolder" (at 184.15 71.12 0)
       (effects (font (size 1.524 1.524)) hide)
     )
@@
       (effects (font (size 1.27 1.27)) (justify left))
     )
-    (property "Footprint" "w_smd_cap:c_2220" (at 231.14 35.56 0)
+    (property "Footprint" "CRF1:c_2220" (at 231.14 35.56 0)
       (effects (font (size 1.524 1.524)) hide)
     )
@@
       (effects (font (size 1.016 1.016)))
     )
-    (property "Footprint" "CRF1:SOT-223" (at 160.02 30.48 0)
+    (property "Footprint" "Package_TO_SOT_SMD:SOT-223" (at 160.02 30.48 0)
       (effects (font (size 1.524 1.524)) hide)
     )
@@
       (effects (font (size 1.016 1.016)))
     )
-    (property "Footprint" "w_smd_diode:do214ac" (at 234.95 54.61 0)
-      (effects (font (size 1.524 1.524)) hide)
-    )
+    (property "Footprint" "CRF1:do214ac" (at 234.95 54.61 0)
+      (effects (font (size 1.524 1.524)) hide)
+    )

Commit message: Final 20230228
Parts:
- U2: footprint Package_TO_SOT_SMD:SOT-223 -> CRF1:SOT-223
Changed lines of the file:
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@@
       (effects (font (size 1.016 1.016)))
     )
-    (property "Footprint" "Package_TO_SOT_SMD:SOT-223" (at 160.02 30.48 0)
+    (property "Footprint" "CRF1:SOT-223" (at 160.02 30.48 0)
       (effects (font (size 1.524 1.524)) hide)
     )
